File: STARBIE W.kicad_pcb (KiCad board)
At the start: 2 copper layers, 101.5 x 99 mm, 6 parts, among them J1 Conn_01x04, J2 Conn_01x08, SW1 SW_Push, SW2 SW_Push, U1 XIAO-ESP32-C3-SMD

Commit message: updated files after some resolved problems
Parts:
- added U2: DHT11, Sensor:Aosong_DHT11_5.5x12.0_P2.54mm, F.Cu at (163.0, 37.0)
- J1: footprint Connector_PinHeader_2.54mm:PinHeader_1x04_P2.54mm_Vertical -> Imported Parts:Display_128x64_096_I2C
- R1: footprint Resistor_THT:R_Axial_DIN0207_L6.3mm_D2.5mm_P10.16mm_Horizontal -> Resistor_THT:R_Axial_DIN0204_L3.6mm_D1.6mm_P7.62mm_Horizontal
- SW1, SW2: footprint Button_Switch_THT:SW_PUSH_6mm -> Button_Switch_Keyboard:SW_Cherry_MX_1.00u_PCB
- U1: footprint RF_Module:MCU_Seeed_ESP32C3 -> Imported Parts:XIAO-ESP32-C3-SMD
- moved R1 64.9 mm to (170.3, 31.0), turned to 180 degrees
- moved J2 47.9 mm to (187.0, 74.8), turned to 0 degrees
- moved SW1 35.9 mm to (135.9, 61.9)
- moved J1 31.7 mm to (165.3, 46.8), turned to 0 degrees
- moved SW2 16.1 mm to (152.5, 84.5)
- moved U1 3.39 mm to (180.5, 71.4)
Routing:
- net +3.3V: track 169.0 -> 115.6 mm, vias 0 -> 2
- net /SDA: track 33.6 -> 75.7 mm, vias 0 -> 1
- net /BTN2: track 25.5 -> 64.2 mm
- net GND: track 113.6 -> 151.8 mm, vias 0 -> 1
- net /DHT: track 55.8 -> 33.3 mm
- net /BTN1: track 74.0 -> 58.6 mm
- net /SCL: track 37.2 -> 41.5 mm
Other:
- board size 101.5 x 99 mm -> 106 x 96.3 mm
