File: STARBIE W.kicad_sch (KiCad schematic)
At the start: 7 parts, among them J1 Conn_01x04, J2 Conn_01x08, SW1 SW_Push, SW2 SW_Push, U1 XIAO-ESP32-C3-SMD, U2 DHT11

Commit message: updated files after some resolved problems
Parts:
- J1: footprint Connector_PinHeader_2.54mm:PinHeader_1x04_P2.54mm_Vertical -> Imported Parts:Display_128x64_096_I2C
- R1: footprint Resistor_THT:R_Axial_DIN0207_L6.3mm_D2.5mm_P10.16mm_Horizontal -> Resistor_THT:R_Axial_DIN0204_L3.6mm_D1.6mm_P7.62mm_Horizontal
- SW1, SW2: footprint Button_Switch_THT:SW_PUSH_6mm -> Button_Switch_Keyboard:SW_Cherry_MX_1.00u_PCB
- U1: footprint RF_Module:MCU_Seeed_ESP32C3 -> Imported Parts:XIAO-ESP32-C3-SMD
Other:
- moved on the sheet: J1
Changed lines of the file:
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@@
 	(wire
 		(pts
-			(xy 187.96 139.7) (xy 187.96 140.97)
+			(xy 190.5 95.25) (xy 190.5 96.52)
 		)
 		(stroke
@@
 	(wire
 		(pts
-			(xy 199.39 146.05) (xy 222.25 146.05)
+			(xy 201.93 101.6) (xy 224.79 101.6)
 		)
 		(stroke
@@
 	(wire
 		(pts
-			(xy 187.96 140.97) (xy 222.25 140.97)
+			(xy 190.5 96.52) (xy 224.79 96.52)
 		)
 		(stroke
@@
 	(wire
 		(pts
-			(xy 194.31 143.51) (xy 222.25 143.51)
+			(xy 196.85 99.06) (xy 224.79 99.06)
 		)
 		(stroke
@@
 	(wire
 		(pts
-			(xy 209.55 148.59) (xy 222.25 148.59)
+			(xy 212.09 104.14) (xy 224.79 104.14)
 		)
 		(stroke
@@
 	)
 	(label "SCL"
-		(at 199.39 146.05 0)
+		(at 201.93 101.6 0)
 		(effects
 			(font
@@
 	)
 	(label "SDA"
-		(at 209.55 148.59 0)
+		(at 212.09 104.14 0)
 		(effects
 			(font
@@
 			)
 		)
-		(property "Footprint" "Button_Switch_THT:SW_PUSH_6mm"
+		(property "Footprint" "Button_Switch_Keyboard:SW_Cherry_MX_1.00u_PCB"
 			(at 63.5 102.87 0)
 			(hide yes)
@@
 			)
 		)
-		(property "Footprint" "Resistor_THT:R_Axial_DIN0207_L6.3mm_D2.5mm_P10.16mm_Horizontal"
+		(property "Footprint" "Resistor_THT:R_Axial_DIN0204_L3.6mm_D1.6mm_P7.62mm_Horizontal"
 			(at 103.632 33.02 90)
 			(hide yes)
@@
 	(symbol
 		(lib_id "Connector_Generic:Conn_01x04")
-		(at 227.33 143.51 0)
+		(at 229.87 99.06 0)
 		(unit 1)
 		(body_style 1)
@@
 		(fields_autoplaced yes)
 		(property "Reference" "J1"
-			(at 229.87 143.5099 0)
+			(at 232.41 99.0599 0)
 			(show_name no)
 			(do_not_autoplace no)
@@
 		)
 		(property "Value" "Conn_01x04"
-			(at 229.87 146.0499 0)
+			(at 232.41 101.5999 0)
 			(show_name no)
 			(do_not_autoplace no)
@@
 			)
 		)
-		(property "Footprint" "Connector_PinHeader_2.54mm:PinHeader_1x04_P2.54mm_Vertical"
-			(at 227.33 143.51 0)
+		(property "Footprint" "Imported Parts:Display_128x64_096_I2C"
+			(at 229.87 99.06 0)
 			(hide yes)
 			(show_name no)
@@
 		)
 		(property "Datasheet" ""
-			(at 227.33 143.51 0)
+			(at 229.87 99.06 0)
 			(hide yes)
 			(show_name no)
@@
 		)
 		(property "Description" "Generic connector, single row, 01x04, script generated (kicad-library-utils/schlib/autogen/connector/)"
-			(at 227.33 143.51 0)
+			(at 229.87 99.06 0)
 			(hide yes)
 			(show_name no)
@@
 			)
 		)
-		(property "Footprint" "RF_Module:MCU_Seeed_ESP32C3"
+		(property "Footprint" "Imported Parts:XIAO-ESP32-C3-SMD"
 			(at 109.982 115.824 0)
 			(hide yes)
@@
 	(symbol
 		(lib_id "power:GND")
-		(at 187.96 139.7 0)
+		(at 190.5 95.25 0)
 		(unit 1)
 		(body_style 1)
@@
 		(fields_autoplaced yes)
 		(property "Reference" "#PWR06"
-			(at 187.96 146.05 0)
+			(at 190.5 101.6 0)
 			(hide yes)
 			(show_name no)
@@
 		)
 		(property "Value" "GND"
-			(at 187.96 144.78 0)
+			(at 190.5 100.33 0)
 			(show_name no)
 			(do_not_autoplace no)
@@
 		)
 		(property "Footprint" ""
-			(at 187.96 139.7 0)
+			(at 190.5 95.25 0)
 			(hide yes)
 			(show_name no)
@@
 		)
 		(property "Datasheet" ""
-			(at 187.96 139.7 0)
+			(at 190.5 95.25 0)
 			(hide yes)
 			(show_name no)
@@
 		)
 		(property "Description" "Power symbol creates a global label with name \"GND\" , ground"
-			(at 187.96 139.7 0)
+			(at 190.5 95.25 0)
 			(hide yes)
 			(show_name no)
@@
 			)
 		)
-		(property "Footprint" "Button_Switch_THT:SW_PUSH_6mm"
+		(property "Footprint" "Button_Switch_Keyboard:SW_Cherry_MX_1.00u_PCB"
 			(at 63.5 78.74 0)
 			(hide yes)
@@
 	(symbol
 		(lib_id "power:+3.3V")
-		(at 194.31 143.51 0)
+		(at 196.85 99.06 0)
 		(unit 1)
 		(body_style 1)
@@
 		(dnp no)
 		(property "Reference" "#PWR07"
-			(at 194.31 147.32 0)
+			(at 196.85 102.87 0)
 			(hide yes)
 			(show_name no)
@@
 		)
 		(property "Value" "+3.3V"
-			(at 198.628 133.35 0)
+			(at 201.168 88.9 0)
 			(hide yes)
 			(show_name no)
@@
 		)
 		(property "Footprint" ""
-			(at 194.31 143.51 0)
+			(at 196.85 99.06 0)
 			(hide yes)
 			(show_name no)
@@
 		)
 		(property "Datasheet" ""
-			(at 194.31 143.51 0)
+			(at 196.85 99.06 0)
 			(hide yes)
 			(show_name no)
@@
 		)
 		(property "Description" "Power symbol creates a global label with name \"+3.3V\""
-			(at 194.31 143.51 0)
-			(hide yes)
-			(show_name no)
+			(at 196.85 99.06 0)
+			(hide yes)
+			(show_name no)
